Commit message: Trying to implement the traditional method

File: resources/task_assets/knob/knob.urdf (robot description, URDF)
Before this commit: robot knob_exp, 4 links, 3 joints
Joints:
- joint actuator_1_joint: limit lower=-1.5707963267948966 upper=3.141592653589793 effort=2 velocity=5 -> lower=0 upper=12.5663706144 effort=2 velocity=5
