Commit message: traditional method completed

File: resources/robots/g1_description/g1_lighter_with_hand_with_contact_force_sensor_traditional.urdf (robot description, URDF)
Before this commit: robot g1_29dof_with_hand, 35 links, 34 joints
Links:
- removed link right_hand_index_1_force_sensor_1_link
- removed link right_hand_index_1_force_sensor_2_link
- removed link right_hand_index_1_force_sensor_3_link
- removed link right_hand_thumb_2_force_sensor_1_link
- removed link right_hand_thumb_2_force_sensor_2_link
- removed link right_hand_thumb_2_force_sensor_3_link
Joints:
- removed joint right_hand_index_1_force_sensor_1_joint
- removed joint right_hand_index_1_force_sensor_2_joint
- removed joint right_hand_index_1_force_sensor_3_joint
- removed joint right_hand_thumb_2_force_sensor_1_joint
- removed joint right_hand_thumb_2_force_sensor_2_joint
- removed joint right_hand_thumb_2_force_sensor_3_joint
