Commit message: Traditional method for the playboard knob task completed!

File: resources/task_assets/playboard/playboard.urdf (robot description, URDF)
Before this commit: robot knob_exp, 10 links, 9 joints
Links:
- link knob_1: geometry collision mesh filename=meshes/knob_1.stl scale=0.001 0.001 0.001; visual mesh filename=meshes/knob_1.stl scale=0.001 0.001 0.001
- link knob_2: geometry collision mesh filename=meshes/knob_2.stl scale=0.001 0.001 0.001; visual mesh filename=meshes/knob_2.stl scale=0.001 0.001 0.001
- link knob_3: geometry collision mesh filename=meshes/knob_3.stl scale=0.001 0.001 0.001; visual mesh filename=meshes/knob_3.stl scale=0.001 0.001 0.001
- link knob_holder_1: geometry collision mesh filename=meshes/knob_holder_1.stl scale=0.001 0.001 0.001; visual mesh filename=meshes/knob_holder_1.stl scale=0.001 0.001 0.001
- link knob_holder_2: geometry collision mesh filename=meshes/knob_holder_2.stl scale=0.001 0.001 0.001; visual mesh filename=meshes/knob_holder_2.stl scale=0.001 0.001 0.001
- link knob_holder_3: geometry collision mesh filename=meshes/knob_holder_3.stl scale=0.001 0.001 0.001; visual mesh filename=meshes/knob_holder_3.stl scale=0.001 0.001 0.001
- link knob_indicator_1: geometry visual box size=0.01 0.0025 0.001
- link knob_indicator_2: geometry visual box size=0.01 0.0025 0.001
- link knob_indicator_3: geometry visual box size=0.01 0.0025 0.001
- link wall_link: geometry collision mesh filename=meshes/wall.stl scale=0.001 0.001 0.001; visual mesh filename=meshes/wall.stl scale=0.001 0.001 0.001
Joints:
- joint knob_1_joint: origin xyz=41 79.62899999999999 365.9124 rpy=0 0 0 -> xyz=0.040999999999999995 0.07962899999999999 0.3659124 rpy=0 0 0
- joint knob_2_joint: origin xyz=27 179.62879999999998 365.9124 rpy=0 0 0 -> xyz=0.027 0.17962879999999998 0.3659124 rpy=0 0 0
- joint knob_3_joint: origin xyz=27 279.6286 365.9124 rpy=0 0 0 -> xyz=0.027 0.27962859999999995 0.3659124 rpy=0 0 0
- joint knob_holder_2_joint: child knob_holder_1 -> knob_holder_2
- joint knob_holder_3_joint: child knob_holder_1 -> knob_holder_3
- joint knob_indicator_1_joint_rigid: origin xyz=5 0 6 rpy=0 0 0 -> xyz=0.005 0 0.006 rpy=0 0 0
- joint knob_indicator_2_joint_rigid: origin xyz=10 12 0 rpy=0 0 0 -> xyz=0.01 0.012 0 rpy=0 0 0
- joint knob_indicator_3_joint_rigid: origin xyz=19 16 0 rpy=0 0 0 -> xyz=0.019 0.016 0 rpy=0 0 0
